File: Hardware/LCR_Meter/current_meter_sch.kicad_sch (KiCad schematic)
At the start: 0 parts

Commit message: work on KCR schematic
Parts:
- added U?: AD620, symbol Amplifier_Instrumentation:AD620
- added U?: AD8610, symbol Amplifier_Operational:AD8610
Changed lines of the file:
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@@
     (effects (font (size 1.27 1.27)) (justify left))
   )
-  (hierarchical_label "I_out" (shape output) (at 125.73 97.79 180)
-    (effects (font (size 1.27 1.27)) (justify right))
-  )
-  (hierarchical_label "I_in" (shape input) (at 125.73 92.71 180)
+  (hierarchical_label "I_in" (shape input) (at 111.76 95.25 180)
     (effects (font (size 1.27 1.27)) (justify right))
   )
@@
     (effects (font (size 1.27 1.27)) (justify left))
   )
+  (symbol (lib_id "Amplifier_Instrumentation:AD620") (at 148.59 119.38 0) (unit 1)
+    (in_bom yes) (on_board yes) (fields_autoplaced)
+    (property "Reference" "U?" (id 0) (at 161.29 114.681 0))
+    (property "Value" "AD620" (id 1) (at 161.29 117.221 0))
+    (property "Footprint" "" (id 2) (at 148.59 119.38 0)
+      (effects (font (size 1.27 1.27)) hide)
+    )
+    (property "Datasheet" "https://www.analog.com/media/en/technical-documentation/data-sheets/AD620.pdf" (id 3) (at 148.59 119.38 0)
+      (effects (font (size 1.27 1.27)) hide)
+    )
+    (pin "1")
+    (pin "2")
+    (pin "3")
+    (pin "4")
+    (pin "5")
+    (pin "6")
+    (pin "7")
+    (pin "8")
+  )
+  (symbol (lib_id "Amplifier_Operational:AD8610") (at 143.51 97.79 0) (unit 1)
+    (in_bom yes) (on_board yes) (fields_autoplaced)
+    (property "Reference" "U?" (id 0) (at 153.67 93.091 0))
+    (property "Value" "AD8610" (id 1) (at 153.67 95.631 0))
+    (property "Footprint" "" (id 2) (at 144.78 96.52 0)
+      (effects (font (size 1.27 1.27)) hide)
+    )
+    (property "Datasheet" "https://www.analog.com/media/en/technical-documentation/data-sheets/AD8610_8620.pdf" (id 3) (at 147.32 93.98 0)
+      (effects (font (size 1.27 1.27)) hide)
+    )
+    (pin "1")
+    (pin "2")
+    (pin "3")
+    (pin "4")
+    (pin "5")
+    (pin "6")
+    (pin "7")
+    (pin "8")
+  )
 )
