File: Hardware/LCR_Meter/voltage_meter_sch.kicad_sch (KiCad schematic)
At the start: 0 parts

Commit message: work on KCR schematic
Parts:
- added U?: AD620, symbol Amplifier_Instrumentation:AD620
- added U?: AD8610, symbol Amplifier_Operational:AD8610
Changed lines of the file:
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@@
     (effects (font (size 1.27 1.27)) (justify left))
   )
+  (symbol (lib_id "Amplifier_Instrumentation:AD620") (at 146.05 138.43 0) (unit 1)
+    (in_bom yes) (on_board yes) (fields_autoplaced)
+    (property "Reference" "U?" (id 0) (at 158.75 133.731 0))
+    (property "Value" "AD620" (id 1) (at 158.75 136.271 0))
+    (property "Footprint" "" (id 2) (at 146.05 138.43 0)
+      (effects (font (size 1.27 1.27)) hide)
+    )
+    (property "Datasheet" "https://www.analog.com/media/en/technical-documentation/data-sheets/AD620.pdf" (id 3) (at 146.05 138.43 0)
+      (effects (font (size 1.27 1.27)) hide)
+    )
+    (pin "1")
+    (pin "2")
+    (pin "3")
+    (pin "4")
+    (pin "5")
+    (pin "6")
+    (pin "7")
+    (pin "8")
+  )
+  (symbol (lib_id "Amplifier_Operational:AD8610") (at 208.28 114.3 0) (unit 1)
+    (in_bom yes) (on_board yes) (fields_autoplaced)
+    (property "Reference" "U?" (id 0) (at 218.44 109.601 0))
+    (property "Value" "AD8610" (id 1) (at 218.44 112.141 0))
+    (property "Footprint" "" (id 2) (at 209.55 113.03 0)
+      (effects (font (size 1.27 1.27)) hide)
+    )
+    (property "Datasheet" "https://www.analog.com/media/en/technical-documentation/data-sheets/AD8610_8620.pdf" (id 3) (at 212.09 110.49 0)
+      (effects (font (size 1.27 1.27)) hide)
+    )
+    (pin "1")
+    (pin "2")
+    (pin "3")
+    (pin "4")
+    (pin "5")
+    (pin "6")
+    (pin "7")
+    (pin "8")
+  )
 )
