File: Hardware/LCR_Meter/zerocrossing_phase_detector_sch.kicad_sch (KiCad schematic)
At the start: 0 parts

Commit message: work on Phase detector
Parts:
- added C? (x4): 100n, Capacitor_SMD:C_0805_2012Metric_Pad1.18x1.45mm_HandSolder, symbol 010_SMD_Capacitors:C_0805_hs
- added R? (x2): 0R, Resistor_SMD:R_1206_3216Metric, symbol 000_SMD_Resitors:R_1206
- added R? (x2): 10k, Resistor_SMD:R_1206_3216Metric, symbol 000_SMD_Resitors:R_1206
- added U? (x6): 74HC74, symbol 74xx:74HC74
- added U? (x5): 74HC86, symbol 74xx:74HC86
- added U? (x2): AD822ARZ, Package_SO:SOIC-8_3.9x4.9mm_P1.27mm, symbol 200_OPAMP:AD822ARZ
- added U? (x2): ADA4860-1, Package_TO_SOT_SMD:SOT-23-6, symbol 200_OPAMP:ADA4860-1
Connections:
- net A: now also U?.3 (+)
- net B: now also U?.3 (+)
- net GND: now also C?.2, C?.2, C?.2, C?.2, U?.10, U?.12, U?.13, U?.4 (-), U?.4 (-), U?.9
- net V+: now also C?.1, C?.1, U?.6 (V+), U?.6 (V+)
- net V-: now also C?.1, C?.1, R?.2, R?.2, U?.2 (V-), U?.2 (V-)
- new net: U?.12 (D), U?.4, U?.5 (Q)
- new net: U?.5, U?.9 (Q)
- new net: R?.1, U?.5 (DISABLE) (x2)
- new net: U?.2 (D), U?.8 (~{Q}) (x2)
- new net: R?.2, U?.11 (C), U?.3 (C) (x2)
- new net: U?.1, U?.9 (Q)
- new net: U?.12 (D), U?.2, U?.5 (Q)
- new net: R?.1, U?.1 (x2)
Other:
- note added: "zero crossing comparator"
