File: Hardware/LCR_Meter/LCR_Meter.kicad_sch (KiCad schematic)
At the start: 4 parts

Commit message: work on signal generator
Other:
- sheet signal_generator ports: added +5V, -5V, EN, SPI_CH_MCP41010, SPI_CS_AD9833; removed SPI_CS, V+, V-
Changed lines of the file:
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@@
     )
   )
-  (sheet (at 120.4722 19.05) (size 31.9278 35.56)
+  (sheet (at 120.65 19.05) (size 31.75 35.56)
     (stroke (width 0.1524) (type solid) (color 0 0 0 0))
     (fill (color 0 0 0 0.0000))
-    (property "Sheet name" "signal_generator" (id 0) (at 120.65 16.2306 0)
+    (property "Sheet name" "signal_generator" (id 0) (at 120.8278 16.2306 0)
       (effects (font (size 1.27 1.27)) (justify left bottom))
     )
-    (property "Sheet file" "signal_generator_sch.kicad_sch" (id 1) (at 120.65 16.2306 0)
+    (property "Sheet file" "signal_generator_sch.kicad_sch" (id 1) (at 120.8278 16.2306 0)
       (effects (font (size 1.27 1.27)) (justify left top))
-    )
-    (pin "V+" input (at 120.4722 43.18 180)
-      (effects (font (size 1.27 1.27)) (justify left))
-    )
-    (pin "V-" output (at 120.4722 45.72 180)
-      (effects (font (size 1.27 1.27)) (justify left))
     )
     (pin "out" output (at 152.4 48.26 0)
@@
       (effects (font (size 1.27 1.27)) (justify left))
     )
-    (pin "SPI_CLK" input (at 120.4722 21.59 180)
-      (effects (font (size 1.27 1.27)) (justify left))
-    )
-    (pin "+3.3V" input (at 120.4722 39.37 180)
-      (effects (font (size 1.27 1.27)) (justify left))
-    )
-    (pin "SPI_MOSI" input (at 120.4722 24.13 180)
-      (effects (font (size 1.27 1.27)) (justify left))
-    )
-    (pin "SPI_CS" input (at 120.4722 26.67 180)
+    (pin "SPI_CLK" input (at 120.65 21.59 180)
+      (effects (font (size 1.27 1.27)) (justify left))
+    )
+    (pin "+3.3V" input (at 120.65 39.37 180)
+      (effects (font (size 1.27 1.27)) (justify left))
+    )
+    (pin "SPI_MOSI" input (at 120.65 24.13 180)
+      (effects (font (size 1.27 1.27)) (justify left))
+    )
+    (pin "SPI_CH_MCP41010" input (at 120.65 26.67 180)
+      (effects (font (size 1.27 1.27)) (justify left))
+    )
+    (pin "SPI_CS_AD9833" input (at 120.65 29.21 180)
+      (effects (font (size 1.27 1.27)) (justify left))
+    )
+    (pin "EN" input (at 120.65 34.29 180)
+      (effects (font (size 1.27 1.27)) (justify left))
+    )
+    (pin "+5V" input (at 120.65 41.91 180)
+      (effects (font (size 1.27 1.27)) (justify left))
+    )
+    (pin "-5V" input (at 120.65 44.45 180)
       (effects (font (size 1.27 1.27)) (justify left))
     )
@@
       (reference "C?") (unit 1) (value "100n") (footprint "Capacitor_SMD:C_1206_3216Metric")
     )
+    (path "/eb72df69-0d7b-45d1-ac9b-f5f7558dee68/0a5640f1-dd42-45f0-b364-47badc4302b9"
+      (reference "C?") (unit 1) (value "4.7u") (footprint "Capacitor_SMD:C_0805_2012Metric_Pad1.18x1.45mm_HandSolder")
+    )
+    (path "/eb72df69-0d7b-45d1-ac9b-f5f7558dee68/0aa9868b-bee9-4c40-94aa-538137622689"
+      (reference "C?") (unit 1) (value "10n") (footprint "Capacitor_SMD:C_0805_2012Metric_Pad1.18x1.45mm_HandSolder")
+    )
     (path "/d1422d36-ee99-4795-804f-b865553c7f13/0bd4f34c-719a-4a2f-9253-4be87b4fffea"
       (reference "C?") (unit 1) (value "100n") (footprint "Capacitor_SMD:C_0805_2012Metric_Pad1.18x1.45mm_HandSolder")
@@
       (reference "C?") (unit 1) (value "100n") (footprint "Capacitor_SMD:C_0805_2012Metric_Pad1.18x1.45mm_HandSolder")
     )
+    (path "/eb72df69-0d7b-45d1-ac9b-f5f7558dee68/8106eac3-2af6-4db2-8949-04036a5dea66"
+      (reference "C?") (unit 1) (value "4.7u") (footprint "Capacitor_SMD:C_0805_2012Metric_Pad1.18x1.45mm_HandSolder")
+    )
+    (path "/eb72df69-0d7b-45d1-ac9b-f5f7558dee68/9110e316-bd9e-4860-8da5-00f28cb07976"
+      (reference "C?") (unit 1) (value "1u") (footprint "Capacitor_SMD:C_0805_2012Metric_Pad1.18x1.45mm_HandSolder")
+    )
+    (path "/eb72df69-0d7b-45d1-ac9b-f5f7558dee68/a5e08701-7c0c-42f0-b214-9921b3714492"
+      (reference "C?") (unit 1) (value "1u") (footprint "Capacitor_SMD:C_0805_2012Metric_Pad1.18x1.45mm_HandSolder")
+    )
     (path "/eb72df69-0d7b-45d1-ac9b-f5f7558dee68/a8d2828f-0704-4481-9cbc-38d29b2ce63b"
       (reference "C?") (unit 1) (value "100n") (footprint "Capacitor_SMD:C_0805_2012Metric_Pad1.18x1.45mm_HandSolder")
@@
       (reference "C?") (unit 1) (value "100n") (footprint "Capacitor_SMD:C_0805_2012Metric_Pad1.18x1.45mm_HandSolder")
     )
-    (path "/eb72df69-0d7b-45d1-ac9b-f5f7558dee68/df7dd165-5ad5-48b5-988d-c6c9838b4a66"
-      (reference "C?") (unit 1) (value "10n") (footprint "Capacitor_SMD:C_0805_2012Metric_Pad1.18x1.45mm_HandSolder")
-    )
     (path "/eb72df69-0d7b-45d1-ac9b-f5f7558dee68/fa6ed327-7524-468a-8671-9fbb7cb3ac69"
       (reference "C?") (unit 1) (value "100n") (footprint "Capacitor_SMD:C_0805_2012Metric_Pad1.18x1.45mm_HandSolder")
@@
       (reference "J?") (unit 1) (value "H_CUR") (footprint "Connector_Coaxial:SMA_Amphenol_132291-12_Vertical")
     )
+    (path "/eb72df69-0d7b-45d1-ac9b-f5f7558dee68/0ad992f0-abf4-4987-a724-64424bbd16b5"
+      (reference "R?") (unit 1) (value "0R") (footprint "Resistor_SMD:R_1206_3216Metric")
+    )
     (path "/3366fbd2-b7c6-4ccb-afdd-03c00c73e9fc/0e2af59b-805c-4b81-a808-8e6d6fd50b52"
       (reference "R?") (unit 1) (value "10k") (footprint "Resistor_SMD:R_1206_3216Metric")
@@
       (reference "R?") (unit 1) (value "10k") (footprint "Resistor_SMD:R_1206_3216Metric")
     )
+    (path "/eb72df69-0d7b-45d1-ac9b-f5f7558dee68/a28a7243-c7c9-4bd6-b759-06ffb8c52403"
+      (reference "R?") (unit 1) (value "910") (footprint "Resistor_SMD:R_1206_3216Metric")
+    )
     (path "/3366fbd2-b7c6-4ccb-afdd-03c00c73e9fc/c6ff8418-6bd5-42c2-8622-1677942dee4e"
       (reference "R?") (unit 1) (value "100") (footprint "Resistor_SMD:R_1206_3216Metric")
@@
       (reference "R?") (unit 1) (value "1k") (footprint "Resistor_SMD:R_1206_3216Metric")
     )
-    (path "/eb72df69-0d7b-45d1-ac9b-f5f7558dee68/072bb016-7b32-4a51-80fd-3a7aad260854"
-      (reference "U?") (unit 1) (value "AD822ARZ") (footprint "Package_SO:SOIC-8_3.9x4.9mm_P1.27mm")
+    (path "/eb72df69-0d7b-45d1-ac9b-f5f7558dee68/6499cb22-393d-4410-a4e4-58593564ba36"
+      (reference "TP?") (unit 1) (value "SigGen") (footprint "")
     )
     (path "/eb72df69-0d7b-45d1-ac9b-f5f7558dee68/11187340-b06f-41a6-87df-8a4ad65837a8"
@@
       (reference "U?") (unit 1) (value "AD8610") (footprint "")
     )
+    (path "/eb72df69-0d7b-45d1-ac9b-f5f7558dee68/d9254451-2f35-499e-85e2-1e7f92b89154"
+      (reference "U?") (unit 1) (value "AD8051ARZ") (footprint "Package_SO:SOIC-8_3.9x4.9mm_P1.27mm")
+    )
     (path "/d1422d36-ee99-4795-804f-b865553c7f13/ef7b66bf-27ef-4f3a-b6ea-10fa66aa73b8"
       (reference "U?") (unit 1) (value "ADA4860-1") (footprint "Package_TO_SOT_SMD:SOT-23-6")
@@
       (reference "U?") (unit 2) (value "74HC74") (footprint "")
     )
+    (path "/eb72df69-0d7b-45d1-ac9b-f5f7558dee68/c9d4029e-bafd-4fd9-b827-a5796b9db0bc"
+      (reference "U?") (unit 2) (value "AD8051ARZ") (footprint "Package_SO:SOIC-8_3.9x4.9mm_P1.27mm")
+    )
     (path "/d1422d36-ee99-4795-804f-b865553c7f13/ebbbeb47-2e32-4ad7-868f-f8c1a55c430b"
       (reference "U?") (unit 2) (value "AD822ARZ") (footprint "Package_SO:SOIC-8_3.9x4.9mm_P1.27mm")
     )
-    (path "/eb72df69-0d7b-45d1-ac9b-f5f7558dee68/ef11a64a-1d9b-4745-8db1-15bc91627311"
-      (reference "U?") (unit 2) (value "AD822ARZ") (footprint "Package_SO:SOIC-8_3.9x4.9mm_P1.27mm")
-    )
